File: MPSIO-Translator.kicad_sch (KiCad schematic)
At the start: 8 parts, among them J1 430451628, J2 430451628, J3 Screw_Terminal_01x02, U1 74LS125

Commit message: Completed Draft of Design
Initial Draft
Parts:
- removed RN1, RN4: 0R, Resistor_SMD:R_Array_Convex_4x1206, symbol Device:R_Pack04
- removed U1: 74LS125, Package_DIP:DIP-14_W7.62mm_Socket_LongPads, symbol 74xx:74LS125
- added C1: 10uF, Capacitor_SMD:C_0805_2012Metric_Pad1.18x1.45mm_HandSolder, symbol Device:C_Small
- added C2: 100nF, Capacitor_SMD:C_0805_2012Metric_Pad1.18x1.45mm_HandSolder, symbol Device:C_Small
- added DRA1, DRA2: 1201578, MountingEquipment:DINRailAdapter_3xM3_PhoenixContact_1201578, symbol Mechanical:DIN_Rail_Adapter
- added U1: 74AHC240, Package_DIP:DIP-20_W7.62mm_Socket_LongPads, symbol 74xx:74AHC240
- J1, J2: footprint (none) -> footprints:430451628; Manufacture (none) -> Molex; Manufacture Part Number (none) -> 0430451628; Supplier (none) -> Digikey; Supplier Part Number (none) -> WM10719-ND
- J3: value Screw_Terminal_01x02 -> Phoenix 1725656; Manufacture (none) -> Phoenix Contact; Manufacture Part Number (none) -> 1725656; Supplier (none) -> Digikey; Supplier Part Number (none) -> 277-1273-ND
- RN1: renamed from RN2; Manufacture (none) -> Panasonic Electronic Components; Manufacture Part Number (none) -> EXB-38V103JV; Supplier (none) -> Digikey; Supplier Part Number (none) -> Y9103CT-ND
- RN2: renamed from RN3; Manufacture (none) -> YAGEO; Manufacture Part Number (none) -> YC164-JR-130RL; Supplier (none) -> Digikey; Supplier Part Number (none) -> 13-YC164-JR-130RLCT-ND
Connections:
- net OUT1_RTN is gone; now on net GND: J1.13
- net OUT2_RTN is gone; now on net GND: J1.14
- net OUT3_RTN is gone; now on net GND: J1.15
- net OUT4_RTN is gone; now on net GND: J1.16
- net GND: now also C1.2, C2.2, U1.1 (1OE), U1.10 (GND), U1.11 (2A3), U1.13 (2A2), U1.15 (2A1), U1.17 (2A0), U1.19 (2OE)
- net OUT1_SRC: now also RN1.4 (R4.1), RN2.8 (R1.2), U1.8 (1A3); no longer RN1.1 (R1.1), RN2.5 (R4.2)
- net OUT1_TRANSLATED: now also RN2.1 (R1.1), U1.12 (1Y3); no longer RN2.4 (R4.1)
- net OUT2_SRC: now also RN1.3 (R3.1), RN2.7 (R2.2), U1.6 (1A2); no longer RN1.2 (R2.1), RN2.6 (R3.2)
- net OUT2_TRANSLATED: now also RN2.2 (R2.1), U1.14 (1Y2); no longer RN2.3 (R3.1)
- net OUT3_SRC: now also RN1.2 (R2.1), RN2.6 (R3.2), U1.4 (1A1); no longer RN1.3 (R3.1), RN2.7 (R2.2)
- net OUT3_TRANSLATED: now also RN2.3 (R3.1), U1.16 (1Y1); no longer RN2.2 (R2.1)
- net OUT4_SRC: now also RN1.1 (R1.1), RN2.5 (R4.2), U1.2 (1A0); no longer RN1.4 (R4.1), RN2.8 (R1.2)
- net OUT4_TRANSLATED: now also RN2.4 (R4.1), U1.18 (1Y0); no longer RN2.1 (R1.1)
- net Vdrive: now also C1.1, C2.1, U1.20 (VCC)
- no-connect marks 0 -> 4
Other:
- note added: "Can Install many Pin-Compatible: SN74*240(Inverting Buffer) or SN74*244 (Non-Inverting Buffer) in the U1 socket. Consider AHC/AC/LVC fmailies for typical 3.3/5V uses"
- note added: "Install RN2 OR U1 NOT BOTH"
- moved on the sheet: J1, J2, J3, RN1, RN2
